File: PCB/starbie.kicad_pcb (KiCad board)
At the start: 2 copper layers, 101.2 x 87 mm, 11 parts, among them J1 Conn_01x04_Pin, J2 Conn_01x08_Pin, J3 Conn_01x02_Pin, SW1 SW_Push, SW2 SW_Push, U1 DHT11, U2 XIAO-ESP32-C3-SMD

Commit message: Edited PCB and BOM
Parts:
- J3: footprint Connector_JST:JST_PH_S2B-PH-SM4-TB_1x02-1MP_P2.00mm_Horizontal -> Connector_JST:JST_XH_S2B-XH-A_1x02_P2.50mm_Horizontal
- R1: footprint Resistor_THT:R_Axial_DIN0204_L3.6mm_D1.6mm_P7.62mm_Horizontal -> Resistor_THT:R_Axial_DIN0207_L6.3mm_D2.5mm_P7.62mm_Horizontal
- moved J3 6.83 mm to (183.6, 119.8)
- moved R1 1.81 mm to (165.8, 56.5)
Routing:
- net /BAT+: track 42.4 -> 36.6 mm
- net GND: track 188.5 -> 183.3 mm
- net /<NO NET>: track 33.1 -> 32.3 mm
- net +3.3V: track 91.0 -> 91.7 mm
